Commit message: update

File: urdf/fake_robot.urdf.xacro (robot description, xacro)
@@ -61,13 +61,12 @@
   <!-- ros2_control -->
   <!-- =============================== -->
-  <ros2_control name="fake_hw_interface::FakeSystem" type="system">
-    <hardware>
-      <!-- 与 plugin xml 中 class 完全一致 -->
+  <!-- <ros2_control name="fake_hw_interface::FakeSystem" type="system"> -->
+    <!-- <hardware>
       <plugin>fake_hw_interface/FakeSystem</plugin>
       <param name="use_mock_hardware" value="$(arg use_mock_hardware)"/>
       <param name="mock_sensor_commands" value="$(arg mock_sensor_commands)"/>
       <param name="slowdown" value="$(arg slowdown)"/>
-    </hardware>
-  <joint name="joint1">
+    </hardware> -->
+  <!-- <joint name="joint1">
     <command_interface name="position"/>
     <state_interface name="position"/>
@@ -83,6 +82,6 @@
     <state_interface name="position"/>
     <state_interface name="velocity"/>
-  </joint>
-  </ros2_control>
+  </joint> -->
+  <!-- </ros2_control> -->
   <ros2_control name="OrinPerceptionSystem" type="system">
   <hardware>
@@ -94,5 +93,5 @@
     <param name="image_width">640</param>
     <param name="image_height">480</param>
-    <param name="framerate">30.0</param>
+    <param name="framerate">60.0</param>
     <param name="pixel_format">mjpeg</param>
     <param name="camera_frame_id">camera_link</param>
